Commit message: add tcp and camera virtual link to the franka urdf

File: franka_panda/panda_with_gripper.urdf (robot description, URDF)
Before this commit: robot panda, 11 links, 10 joints
Links:
- added link camera_link, mass 0.2; visual box size=.08 .025 0.01
- added link tcp_link, mass 0.00001
Joints:
- added joint camera_joint: type fixed, parent panda_hand, child camera_link, origin xyz=-0.05 0 0 rpy=1.3  0 -1.57
- added joint tcp_joint: type fixed, parent panda_hand, child tcp_link, origin xyz=0 0 0.1 rpy=0 0 3.14

Commit message: newton: Update Franka Newton driver and URDF
Improve joint command handling with step limiting for smoother motion.
Add gripper position feedback and fix collision geometry for
hydroelastic contacts in the URDF.

File: franka_panda/panda_with_gripper.urdf (robot description, URDF)
Before this commit: robot panda, 11 links, 10 joints
Links:
- link panda_leftfinger: geometry collision box size=0.02 0.015 0.05; visual mesh filename=meshes/visual/finger.stl
- link panda_rightfinger: geometry collision box size=0.02 0.015 0.05; visual mesh filename=meshes/visual/finger.stl
Joints:
- joint panda_finger_joint1: limit lower=0.0 upper=0.04 effort=20 velocity=0.2 -> lower=0.0 upper=0.04 effort=100 velocity=0.2
- joint panda_finger_joint2: limit lower=0.0 upper=0.04 effort=20 velocity=0.2 -> lower=0.0 upper=0.04 effort=100 velocity=0.2; mimic joint=panda_finger_joint1 -> (none)
